File: Main/NoiseCre.kicad_pcb (KiCad board)
At the start: 2 copper layers, 46 x 116 mm, 53 parts, among them J3 Conn_01x06, Q1 BC548, Q2 2N3906, Q3 2N3906, SW1 SW_DPDT_x2, U1 TL072, U2 LM13700

Commit message: Updated gain output
Parts:
- added C13: 1uF, Capacitor_THT:C_Rect_L7.2mm_W5.5mm_P5.00mm_FKS2_FKP2_MKS2_MKP2, F.Cu at (118.5, 165.0)
- added R28: 6.8K, AO_tht:R_Axial_DIN0207_L6.3mm_D2.5mm_P10.16mm_Horizontal, F.Cu at (126.0, 145.6)
- added R29: 100K, AO_tht:R_Axial_DIN0207_L6.3mm_D2.5mm_P10.16mm_Horizontal, F.Cu at (115.9, 140.8)
- added R30: 100K, AO_tht:R_Axial_DIN0207_L6.3mm_D2.5mm_P10.16mm_Horizontal, F.Cu at (126.0, 160.0)
- U1: value TL072 -> TL074; footprint AO_tht:DIP-8_W7.62mm_Socket_LongPads -> AO_tht:DIP-14_W7.62mm_Socket_LongPads
- moved C10 24.7 mm to (97.5, 139.8), turned to -90 degrees
- moved C11 15.7 mm to (114.5, 133.8), turned to -90 degrees
- moved C6 13.0 mm to (97.9, 147.6), turned to -90 degrees
- moved R25 12.4 mm to (115.9, 155.2)
- moved R13 10.5 mm to (126.0, 150.4), turned to 180 degrees
- moved C7 10.4 mm to (112.3, 150.0), turned to 90 degrees
- moved R2 8.38 mm to (126.0, 129.4)
- moved U1 4.15 mm to (101.3, 140.0)
- moved C1 3.41 mm to (123.5, 134.4)
- moved R27 1.42 mm to (115.9, 176.2)
- moved R9 1.39 mm to (115.9, 171.2)
- moved Q1 1.00 mm to (118.2, 124.0)
- moved C12 0.50 mm to (112.2, 101.9)
- moved C8 0.50 mm to (112.2, 106.8)
- moved C9 0.50 mm to (97.8, 110.0)
Connections:
- net Net-(SW1A-A) renamed Noise
- C10 pad 2: Net-(C10-Pad2) -> Net-(U1C-+)
- R9 pad 2: Net-(C10-Pad2) -> Net-(R29-Pad2)
- U1 pad 4: -12V -> +12V
- U1 pad 8: +12V -> Net-(U1C--)
Routing:
- net Net-(R29-Pad2): track 0.00 -> 49.1 mm
- net Net-(U1D-+): track 0.00 -> 30.0 mm
- net Net-(C10-Pad1): track 69.7 -> 43.5 mm
- net Net-(C10-Pad2): track 18.1 -> 0.00 mm
- net Net-(U1C--): track 0.00 -> 16.9 mm
- net Net-(U1B--): track 12.7 -> 28.8 mm
- net Net-(C11-Pad1): track 54.5 -> 39.6 mm
- net Net-(U1C-+): track 0.00 -> 13.7 mm, vias 0 -> 1
- net Res: track 18.4 -> 31.3 mm, vias 0 -> 1
- net Net-(U1D--): track 0.00 -> 12.5 mm
- net GND: track 29.0 -> 18.7 mm, vias 2 -> 0
- net +12V: track 177.9 -> 168.9 mm, vias 1 -> 0
- net -12V: track 120.2 -> 125.8 mm, vias 0 -> 1
- net Net-(U1A--): track 64.7 -> 60.4 mm
- net Net-(Q1-E): track 14.4 -> 17.9 mm
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